Commit message: mine gripper

File: urdf/binpicking_gripper_macro.xacro (robot description, xacro)
@@ -2,5 +2,5 @@
 <robot
     xmlns:xacro="http://ros.org/wiki/xacro">
-    <xacro:property name="length" value="0.173" />
+    <xacro:property name="length" value="0.166" />
     <xacro:property name="radius1" value="0.020" />
     <xacro:property name="radius2" value="0.007" />
@@ -9,7 +9,8 @@
         <link name="${prefix}base_link">
             <visual>
-                <origin rpy="0 0 0" xyz="-0.00250 -0.03750 -0.03750" />
+                <!-- <origin rpy="0 0 0" xyz="0 0 0" /> -->
+                <origin rpy="0 ${pi/2} 0" xyz="0 -0.035 0.035" />
                 <geometry>
-                    <mesh filename="package://bin_picking/meshes/gripper.stl" />
+                    <mesh filename="package://bin_picking/meshes/gripper.STL" />
                 </geometry>
                 <material name="">
@@ -20,5 +21,5 @@
                 <!-- <origin rpy="0 0 0" xyz="-0.16250 -0.03750 -0.03750"/> -->
                 <geometry>
-                    <mesh filename="package://bin_picking/meshes/gripper.stl" />
+                    <mesh filename="package://bin_picking/meshes/gripper.STL" />
                 </geometry>
             </collision>
