Commit message: calibration of the laser sensor

File: bin_picking/urdf/binpicking_robot_macro.xacro (robot description, xacro)
@@ -7,4 +7,6 @@
     <!-- include end effector gripper -->
     <xacro:include filename="$(find bin_picking)/urdf/binpicking_gripper_macro.xacro"/>
+    <!-- include laser sensor -->
+    <xacro:include filename="$(find bin_picking)/urdf/binpicking_sensor_macro.xacro"/>
     <!-- manipulator macro -->
     <xacro:macro name="bin_picking_manipulator" params="prefix">
@@ -14,9 +16,16 @@
         <xacro:bin_picking_gripper prefix="${prefix}eef_" />
         <!-- joint connecting the lrmate200id to the end effector -->
-        <joint name="${prefix}robot_flange-${prefix}gripper_base_link" type="fixed">
+        <joint name="${prefix}robot_flange-${prefix}eef_base_link" type="fixed">
             <origin xyz="0 0 0" rpy="0 0 0" />
             <parent link="${prefix}robot_flange" />
             <child link="${prefix}eef_base_link" />
         </joint>
+        <!-- laser sensor -->
+        <xacro:bin_picking_sensor prefix="${prefix}ls_" />
+        <joint name="${prefix}eef_tool_tip-${prefix}ls_base_link" type="fixed">
+            <origin xyz="0.047 0.0166 -0.0636" rpy="0 0 0" />
+            <parent link="${prefix}eef_tool_tip" />
+            <child link="${prefix}ls_base_link" />
+        </joint>
     </xacro:macro>
 </robot>

Commit message: some changes in the camera_calibration_client.py

File: bin_picking/urdf/binpicking_robot_macro.xacro (robot description, xacro)
@@ -24,5 +24,5 @@
         <xacro:bin_picking_sensor prefix="${prefix}ls_" />
         <joint name="${prefix}eef_tool_tip-${prefix}ls_base_link" type="fixed">
-            <origin xyz="0.047 0.0166 -0.0636" rpy="0 0 0" />
+            <origin xyz="0.0478 0.0166 -0.0636" rpy="0 0 0" />
             <parent link="${prefix}eef_tool_tip" />
             <child link="${prefix}ls_base_link" />
