Commit message: kinect calibration close enough

File: bin_picking/urdf/binpicking_macro.xacro (robot description, xacro)
@@ -10,8 +10,11 @@
     <xacro:macro name="bin_picking" params="prefix">
         <xacro:bin_picking_manipulator prefix="${prefix}" />
-        <xacro:kinect_camera name="camera" parent="${prefix}robot_base_link">
+        <xacro:kinect_camera name="camera" parent="${prefix}robot_link_4">
+            <!-- <origin
+                xyz="0.68335329 -0.1191058 1.03896683"
+                rpy="3.0303556  1.7643787 -0.0945628" /> -->
             <origin
-                xyz="0.68335329 -0.1191058 1.03896683"
-                rpy="3.0303556  1.7643787 -0.0945628" />
+                xyz="0.248546721125 0.0815121571909 -0.00896883288009"
+                rpy="-1.5638335 0.1423606 1.5261973" />
         </xacro:kinect_camera>
     </xacro:macro>

Commit message: correct calibration of the Kinect

File: bin_picking/urdf/binpicking_macro.xacro (robot description, xacro)
@@ -11,10 +11,24 @@
         <xacro:bin_picking_manipulator prefix="${prefix}" />
         <xacro:kinect_camera name="camera" parent="${prefix}robot_link_4">
+            <!-- bernardo -->
             <!-- <origin
                 xyz="0.68335329 -0.1191058 1.03896683"
                 rpy="3.0303556  1.7643787 -0.0945628" /> -->
+            <!-- joana 1 -->
+            <!-- <origin
+                xyz="0.248546721125 0.0815121571909 -0.00896883288009"
+                rpy="-1.5638335 0.1423606 1.5261973" /> -->
+            <!-- joana XYZ com Y e Z trocados -->
+            <!-- <origin
+                xyz="0.278189529766 0.113729970677 -0.0189680751133"
+                rpy="-1.5683314 1.5864961 0.0279292" /> -->
+            <!-- joana XYZ -->
+            <!-- <origin
+                xyz="0.278189529766 0.113729970677 -0.0189680751133"
+                rpy="-1.5683314 0.0279292 1.5864961" /> -->
+             <!-- joana convert euler_from_quaternion -->
             <origin
-                xyz="0.248546721125 0.0815121571909 -0.00896883288009"
-                rpy="-1.5638335 0.1423606 1.5261973" />
+                xyz="0.273824339688 0.11318137131 -0.0197138711695"
+                rpy="1.43637243915 1.55845880529 2.99165474735" />
         </xacro:kinect_camera>
     </xacro:macro>

Commit message: new calibration

File: bin_picking/urdf/binpicking_macro.xacro (robot description, xacro)
@@ -11,24 +11,12 @@
         <xacro:bin_picking_manipulator prefix="${prefix}" />
         <xacro:kinect_camera name="camera" parent="${prefix}robot_link_4">
-            <!-- bernardo -->
+             <!-- joana convert euler_from_quaternion 1-->
             <!-- <origin
-                xyz="0.68335329 -0.1191058 1.03896683"
-                rpy="3.0303556  1.7643787 -0.0945628" /> -->
-            <!-- joana 1 -->
-            <!-- <origin
-                xyz="0.248546721125 0.0815121571909 -0.00896883288009"
-                rpy="-1.5638335 0.1423606 1.5261973" /> -->
-            <!-- joana XYZ com Y e Z trocados -->
-            <!-- <origin
-                xyz="0.278189529766 0.113729970677 -0.0189680751133"
-                rpy="-1.5683314 1.5864961 0.0279292" /> -->
-            <!-- joana XYZ -->
-            <!-- <origin
-                xyz="0.278189529766 0.113729970677 -0.0189680751133"
-                rpy="-1.5683314 0.0279292 1.5864961" /> -->
-             <!-- joana convert euler_from_quaternion -->
+                xyz="0.273824339688 0.11318137131 -0.0197138711695"
+                rpy="1.43637243915 1.55845880529 2.99165474735" /> -->
+             <!-- joana convert euler_from_quaternion 2-->
             <origin
-                xyz="0.273824339688 0.11318137131 -0.0197138711695"
-                rpy="1.43637243915 1.55845880529 2.99165474735" />
+                xyz="0.287897942007 0.113658162424 -0.0172542425314"
+                rpy="1.30973391552 1.5275728369 2.88949861591" />
         </xacro:kinect_camera>
     </xacro:macro>

Commit message: Kinect calibration problems and sensor RS232

File: bin_picking/urdf/binpicking_macro.xacro (robot description, xacro)
@@ -11,12 +11,111 @@
         <xacro:bin_picking_manipulator prefix="${prefix}" />
         <xacro:kinect_camera name="camera" parent="${prefix}robot_link_4">
-             <!-- joana convert euler_from_quaternion 1-->
+             <!-- joana convert euler_from_quaternion 1 x para a frente melhor em y-->
             <!-- <origin
                 xyz="0.273824339688 0.11318137131 -0.0197138711695"
                 rpy="1.43637243915 1.55845880529 2.99165474735" /> -->
+            <!-- <origin
+                xyz="0.253824339688 0.11318137131 -0.0197138711695"
+                rpy="1.43637243915 1.55845880529 2.99165474735" /> -->
              <!-- joana convert euler_from_quaternion 2-->
+            <!-- <origin
+                xyz="0.287897942007 0.113658162424 -0.0172542425314"
+                rpy="1.30973391552 1.5275728369 2.88949861591" /> -->
+             <!-- joana convert euler_from_quaternion 3-->
+            <!-- <origin
+                xyz="0.279609095669 0.116639748561 -0.0214942133212"
+                rpy="1.92575936385 1.54891520166 -2.79157664793" /> -->
+             <!-- joana convert euler_from_quaternion 4-->
+            <!-- <origin
+                xyz="0.268440466484 0.122899970085 -0.0166416582814"
+                rpy="2.06885061027 1.55781252086 -2.64482979539" /> -->
+             <!-- joana convert euler_from_quaternion 5 noite x para tras-->
+            <!-- <origin
+                xyz="0.247839774882 0.11700204948 -0.0190325324095"
+                rpy="1.7398943203 1.54554241269 -2.98878736842" /> -->
+             <!-- joana convert euler_from_quaternion 6 noite-->
+            <!-- <origin
+                xyz="0.230029470617 0.132857372442 -0.00630274821251"
+                rpy="2.73368395102 1.54572900105 -1.94362403975" /> -->
+             <!-- joana convert euler_from_quaternion 7 manha-->
+            <!-- <origin
+                xyz="0.276754546937 0.120140773748 -0.0143116801325"
+                rpy="2.1200457846 1.54862201713 -2.59894915819" /> -->
+             <!-- joana convert euler_from_quaternion 8 Miguel BOM x tarde-->
+            <!-- <origin
+                xyz="0.251399988337 0.121134021845 -0.0214740394396"
+                rpy="2.77817146391 1.54118595996 -1.97217228011" /> -->
+             <!-- joana convert euler_from_quaternion 9 MAL tarde-->
+            <!-- <origin
+                xyz="0.290023777948 0.117765053501 -0.0224434855418"
+                rpy="1.76699764666 1.54179041055 -2.95878204774" /> -->
+             <!-- joana convert euler_from_quaternion 10 tarde-->
+            <!-- <origin
+                xyz="0.243917673784 0.131550407348 -0.0194209143795"
+                rpy="2.53224846805 1.54202866651 -2.18035254058" /> -->
+             <!-- joana convert euler_from_quaternion 10 batota-->
+            <!-- <origin
+                xyz="0.251399988337 0.11318137131 -0.0194209143795"
+                rpy="2.53224846805 1.54202866651 -2.18035254058" /> -->
+             <!-- joana convert euler_from_quaternion 11 -->
+            <!-- <origin
+                xyz="0.279007993329 0.117180125822 -0.0180197530052"
+                rpy="1.85013384122 1.54604862537 -2.87502917486" /> -->
+             <!-- joana convert euler_from_quaternion 12 noite -->
+            <!-- <origin
+                xyz="0.2766913732440 0.117286498686 -0.0215517328186"
+                rpy="1.79512358539 1.5416251848 -2.91911484011" /> -->
+             <!-- joana convert euler_from_quaternion 12 noite batota-->
+            <!-- <origin
+                xyz="0.268440466484 0.11318137131 -0.0215517328186"
+                rpy="1.79512358539 1.5416251848 -2.91911484011" /> -->
+             <!-- joana convert euler_from_quaternion 13 noite -->
+            <!-- <origin
+                xyz="0.281486400201 0.116789579978 -0.0224725143874"
+                rpy="1.76283050436 1.54019722186 -2.95054985582" /> -->
+             <!-- joana convert euler_from_quaternion 14 tarde novo aruco
+              -->
+            <!-- <origin
+                xyz="0.280370462232 0.118270345592 -0.0206941993316"
+                rpy="1.8562358457 1.54143707136 -2.86492619894" /> -->
+             <!-- joana convert euler_from_quaternion 15 tarde novo aruco
+              -->
+            <!-- <origin
+                xyz="0.28051830155 0.115758504585 -0.0209927386866"
+                rpy="1.72006698037 1.54206660591 -3.01004459736" /> -->
+             <!-- joana convert euler_from_quaternion 16 tarde novo aruco
+              -->
+            <!-- <origin
+                xyz="0.281981481279 0.11258785627 -0.0175115497053"
+                rpy="1.61898424936 1.5365298456 -3.11537802718" /> -->
+             <!-- joana convert euler_from_quaternion 17 tarde novo aruco poucas frames
+              -->
+            <!-- <origin
+                xyz="0.227161205497 0.128223892751 -0.00633328587159"
+                rpy="2.27333984837 1.54142755852 -2.43197482131" /> -->
+             <!-- joana convert euler_from_quaternion 18 tarde novo aruco 37 frames
+              -->
+            <!-- <origin
+                xyz="0.278978061288 0.116770357766 -0.0210383040274"
+                rpy="1.77711753615 1.54389413149 -2.94693274648" /> -->
+             <!-- joana convert euler_from_quaternion 19 tarde novo aruco 20 frames
+              -->
+            <!-- <origin
+                xyz="0.245273053545 0.117932415176 -0.0189283710983"
+                rpy="1.85016499124 1.54239294719 -2.86964920284" /> -->
+             <!-- joana convert euler_from_quaternion 20 tarde novo aruco 30 frames
+              -->
+            <!-- <origin
+                xyz="0.277881243837 0.119542350176 -0.0206221311455"
+                rpy="1.96078880682 1.54318442414 -2.75917553374" /> -->
+             <!-- joana convert euler_from_quaternion 20 tarde novo aruco 30 frames
+              -->
             <origin
-                xyz="0.287897942007 0.113658162424 -0.0172542425314"
-                rpy="1.30973391552 1.5275728369 2.88949861591" />
+                xyz="0.279403937965 0.129221579884 -0.0219581389451"
+                rpy="2.22624342566 1.53976899344 -2.50437731141" />
+                <!--
+                X entre 0.268440466484 e 0.251399988337
+                Y entre 0.117286498686 e 0.11318137131
+                 -->
         </xacro:kinect_camera>
     </xacro:macro>

Commit message: Kinect Calibration almost perfect

File: bin_picking/urdf/binpicking_macro.xacro (robot description, xacro)
@@ -111,7 +111,22 @@
              <!-- joana convert euler_from_quaternion 20 tarde novo aruco 30 frames
               -->
+            <!-- <origin
+                xyz="0.279403937965 0.129221579884 -0.0219581389451"
+                rpy="2.22624342566 1.53976899344 -2.50437731141" /> -->
+             <!-- joana convert euler_from_quaternion 21 after intrisic calibration GOOD X NOT SO GOOD Y
+              -->
+            <!-- <origin
+                xyz="0.247998706401 0.125155606229 -0.0186859903171"
+                rpy="2.05453674488 1.54706375547 -2.66341374452" /> -->
+             <!-- joana convert euler_from_quaternion 22 after intrisic calibration GOOD X WORST Y
+              -->
+            <!-- <origin
+                xyz="0.245630132675 0.128734721091 -0.0186468780284"
+                rpy="2.18202977374 1.5453374847 -2.52414462864" /> -->
+             <!-- joana convert euler_from_quaternion 23 after intrisic calibration
+              -->
             <origin
-                xyz="0.279403937965 0.129221579884 -0.0219581389451"
-                rpy="2.22624342566 1.53976899344 -2.50437731141" />
+                xyz="0.250037605295 0.121920055033 -0.0198234097631"
+                rpy="1.86250666619 1.54643427609 -2.85870201824" />
                 <!--
                 X entre 0.268440466484 e 0.251399988337

Commit message: pointTFtransfer detect all necessary points

File: bin_picking/urdf/binpicking_macro.xacro (robot description, xacro)
@@ -114,22 +114,75 @@
                 xyz="0.279403937965 0.129221579884 -0.0219581389451"
                 rpy="2.22624342566 1.53976899344 -2.50437731141" /> -->
-             <!-- joana convert euler_from_quaternion 21 after intrisic calibration GOOD X NOT SO GOOD Y
+             <!-- joana convert euler_from_quaternion 21 after intrisic calibration BAD in X
               -->
             <!-- <origin
                 xyz="0.247998706401 0.125155606229 -0.0186859903171"
                 rpy="2.05453674488 1.54706375547 -2.66341374452" /> -->
-             <!-- joana convert euler_from_quaternion 22 after intrisic calibration GOOD X WORST Y
+             <!-- joana convert euler_from_quaternion 22 after intrisic calibration NOT BAD IN BOUTH x: 0.333202 y: 0.192976
               -->
             <!-- <origin
                 xyz="0.245630132675 0.128734721091 -0.0186468780284"
                 rpy="2.18202977374 1.5453374847 -2.52414462864" /> -->
-             <!-- joana convert euler_from_quaternion 23 after intrisic calibration
+             <!-- joana convert euler_from_quaternion 23 after intrisic calibration NOT BAD IN X
               -->
+            <!-- <origin
+                xyz="0.250037605295 0.121920055033 -0.0198234097631"
+                rpy="1.86250666619 1.54643427609 -2.85870201824" /> -->
+             <!-- joana convert euler_from_quaternion 24 after intrisic calibration BEST ONE SO FAR i Y x: 0.337196  y: 0.190538
+              -->
+            <!-- <origin
+                xyz="0.249315737631 0.122836898871 -0.0173595499696"
+                rpy="1.94636293657 1.54585698373 -2.77753500665" /> -->
+             <!-- joana convert euler_from_quaternion 25 after intrisic calibration BAD In X
+              -->
+            <!-- <origin
+                xyz="0.2464362228 0.123022494194 -0.0186746162559"
+                rpy="1.94060142493 1.55129148344 -2.77733685521" /> -->
+             <!-- joana convert euler_from_quaternion 26 after intrisic calibration x: 0.333624  y: 0.193778
+              -->
+            <!-- <origin
+                xyz="0.279827354527 0.12116330125 -0.0182204436316"
+                rpy="1.78482730575 1.55059462639 -2.93123755032" /> -->
+             <!-- joana convert euler_from_quaternion 27 after intrisic calibration x: 0.33612 y: 0.191305
+              -->
+            <!-- <origin
+                xyz="0.247888432512 0.123172523076 -0.0197941758473"
+                rpy="1.90546337967 1.55051949778 -2.80537480944" /> -->
+             <!-- joana convert euler_from_quaternion 28 after intrisic calibration x: 0.333241 y: 0.191324 BEST SO FAR
+              -->
+            <!-- <origin
+                xyz="0.244316235557 0.128274081521 -0.0171762659762"
+                rpy="2.20778889637 1.54928707453 -2.49841856116" /> -->
+             <!-- joana convert euler_from_quaternion 29 after intrisic calibration BAD x: 0.305953 y: 0.19183
+              -->
+            <!-- <origin
+                xyz="0.24973940062 0.122363137841 -0.0173974204673"
+                rpy="1.95908118839 1.54394351042 -2.77092726247" /> -->
+             <!-- joana convert euler_from_quaternion 30 after intrisic calibration SOOO BAD x: 0.366387 y: 0.195049
+              -->
+            <!-- <origin
+                xyz="0.27831321288 0.125011986708 -0.0184730486361"
+                rpy="2.0482106047 1.54868496736 -2.65998966417" /> -->
+             <!-- joana convert euler_from_quaternion 31 after intrisic calibration SOOO x: 0.337417  y: 0.190311
+              -->
+            <!-- <origin
+                xyz="0.248760043608 0.120732900165 -0.0200442441181"
+                rpy="1.8905007158 1.54731656982 -2.84068026775" /> -->
+                <!-- x: 0.333534  y: 0.190602 -->
+<!-- x: 0.332586 y: 0.190537 -->
+            <!-- <origin
+                xyz="0.245460043608 0.120032900165 -0.0200442441181"
+                rpy="1.8905007158 1.54731656982 -2.84068026775" /> -->
+             <!-- After Visions class X verry good x:0.330293 Y BAD y:0.199388    -->
+            <!-- <origin
+                xyz="0.247595042515 0.119885890773 -0.020976224609"
+                rpy="-1.16471837775 1.56523311718 0.4010175495" /> -->
+             <!-- After Visions class X verry good x:0.330293 Y BAD y:0.199388    -->
             <origin
-                xyz="0.250037605295 0.121920055033 -0.0198234097631"
-                rpy="1.86250666619 1.54643427609 -2.85870201824" />
+                xyz="0.247469111314 0.121665921033 -0.0209441353601"
+                rpy="-1.73229551223 1.56538317963 -0.168783829812" />
                 <!--
-                X entre 0.268440466484 e 0.251399988337
-                Y entre 0.117286498686 e 0.11318137131
+                X pouco menor 0.247998706401
+                Y menor 0.121920055033
                  -->
         </xacro:kinect_camera>
