Commit message: correct moveit package

File: bin_picking/urdf/binpicking_macro.xacro (robot description, xacro)
@@ -11,167 +11,4 @@
         <xacro:bin_picking_manipulator prefix="${prefix}" />
         <xacro:kinect_camera name="camera" parent="${prefix}robot_link_4">
-             <!-- joana convert euler_from_quaternion 1 x para a frente melhor em y-->
-            <!-- <origin
-                xyz="0.273824339688 0.11318137131 -0.0197138711695"
-                rpy="1.43637243915 1.55845880529 2.99165474735" /> -->
-            <!-- <origin
-                xyz="0.253824339688 0.11318137131 -0.0197138711695"
-                rpy="1.43637243915 1.55845880529 2.99165474735" /> -->
-             <!-- joana convert euler_from_quaternion 2-->
-            <!-- <origin
-                xyz="0.287897942007 0.113658162424 -0.0172542425314"
-                rpy="1.30973391552 1.5275728369 2.88949861591" /> -->
-             <!-- joana convert euler_from_quaternion 3-->
-            <!-- <origin
-                xyz="0.279609095669 0.116639748561 -0.0214942133212"
-                rpy="1.92575936385 1.54891520166 -2.79157664793" /> -->
-             <!-- joana convert euler_from_quaternion 4-->
-            <!-- <origin
-                xyz="0.268440466484 0.122899970085 -0.0166416582814"
-                rpy="2.06885061027 1.55781252086 -2.64482979539" /> -->
-             <!-- joana convert euler_from_quaternion 5 noite x para tras-->
-            <!-- <origin
-                xyz="0.247839774882 0.11700204948 -0.0190325324095"
-                rpy="1.7398943203 1.54554241269 -2.98878736842" /> -->
-             <!-- joana convert euler_from_quaternion 6 noite-->
-            <!-- <origin
-                xyz="0.230029470617 0.132857372442 -0.00630274821251"
-                rpy="2.73368395102 1.54572900105 -1.94362403975" /> -->
-             <!-- joana convert euler_from_quaternion 7 manha-->
-            <!-- <origin
-                xyz="0.276754546937 0.120140773748 -0.0143116801325"
-                rpy="2.1200457846 1.54862201713 -2.59894915819" /> -->
-             <!-- joana convert euler_from_quaternion 8 Miguel BOM x tarde-->
-            <!-- <origin
-                xyz="0.251399988337 0.121134021845 -0.0214740394396"
-                rpy="2.77817146391 1.54118595996 -1.97217228011" /> -->
-             <!-- joana convert euler_from_quaternion 9 MAL tarde-->
-            <!-- <origin
-                xyz="0.290023777948 0.117765053501 -0.0224434855418"
-                rpy="1.76699764666 1.54179041055 -2.95878204774" /> -->
-             <!-- joana convert euler_from_quaternion 10 tarde-->
-            <!-- <origin
-                xyz="0.243917673784 0.131550407348 -0.0194209143795"
-                rpy="2.53224846805 1.54202866651 -2.18035254058" /> -->
-             <!-- joana convert euler_from_quaternion 10 batota-->
-            <!-- <origin
-                xyz="0.251399988337 0.11318137131 -0.0194209143795"
-                rpy="2.53224846805 1.54202866651 -2.18035254058" /> -->
-             <!-- joana convert euler_from_quaternion 11 -->
-            <!-- <origin
-                xyz="0.279007993329 0.117180125822 -0.0180197530052"
-                rpy="1.85013384122 1.54604862537 -2.87502917486" /> -->
-             <!-- joana convert euler_from_quaternion 12 noite -->
-            <!-- <origin
-                xyz="0.2766913732440 0.117286498686 -0.0215517328186"
-                rpy="1.79512358539 1.5416251848 -2.91911484011" /> -->
-             <!-- joana convert euler_from_quaternion 12 noite batota-->
-            <!-- <origin
-                xyz="0.268440466484 0.11318137131 -0.0215517328186"
-                rpy="1.79512358539 1.5416251848 -2.91911484011" /> -->
-             <!-- joana convert euler_from_quaternion 13 noite -->
-            <!-- <origin
-                xyz="0.281486400201 0.116789579978 -0.0224725143874"
-                rpy="1.76283050436 1.54019722186 -2.95054985582" /> -->
-             <!-- joana convert euler_from_quaternion 14 tarde novo aruco
-              -->
-            <!-- <origin
-                xyz="0.280370462232 0.118270345592 -0.0206941993316"
-                rpy="1.8562358457 1.54143707136 -2.86492619894" /> -->
-             <!-- joana convert euler_from_quaternion 15 tarde novo aruco
-              -->
-            <!-- <origin
-                xyz="0.28051830155 0.115758504585 -0.0209927386866"
-                rpy="1.72006698037 1.54206660591 -3.01004459736" /> -->
-             <!-- joana convert euler_from_quaternion 16 tarde novo aruco
-              -->
-            <!-- <origin
-                xyz="0.281981481279 0.11258785627 -0.0175115497053"
-                rpy="1.61898424936 1.5365298456 -3.11537802718" /> -->
-             <!-- joana convert euler_from_quaternion 17 tarde novo aruco poucas frames
-              -->
-            <!-- <origin
-                xyz="0.227161205497 0.128223892751 -0.00633328587159"
-                rpy="2.27333984837 1.54142755852 -2.43197482131" /> -->
-             <!-- joana convert euler_from_quaternion 18 tarde novo aruco 37 frames
-              -->
-            <!-- <origin
-                xyz="0.278978061288 0.116770357766 -0.0210383040274"
-                rpy="1.77711753615 1.54389413149 -2.94693274648" /> -->
-             <!-- joana convert euler_from_quaternion 19 tarde novo aruco 20 frames
-              -->
-            <!-- <origin
-                xyz="0.245273053545 0.117932415176 -0.0189283710983"
-                rpy="1.85016499124 1.54239294719 -2.86964920284" /> -->
-             <!-- joana convert euler_from_quaternion 20 tarde novo aruco 30 frames
-              -->
-            <!-- <origin
-                xyz="0.277881243837 0.119542350176 -0.0206221311455"
-                rpy="1.96078880682 1.54318442414 -2.75917553374" /> -->
-             <!-- joana convert euler_from_quaternion 20 tarde novo aruco 30 frames
-              -->
-            <!-- <origin
-                xyz="0.279403937965 0.129221579884 -0.0219581389451"
-                rpy="2.22624342566 1.53976899344 -2.50437731141" /> -->
-             <!-- joana convert euler_from_quaternion 21 after intrisic calibration BAD in X
-              -->
-            <!-- <origin
-                xyz="0.247998706401 0.125155606229 -0.0186859903171"
-                rpy="2.05453674488 1.54706375547 -2.66341374452" /> -->
-             <!-- joana convert euler_from_quaternion 22 after intrisic calibration NOT BAD IN BOUTH x: 0.333202 y: 0.192976
-              -->
-            <!-- <origin
-                xyz="0.245630132675 0.128734721091 -0.0186468780284"
-                rpy="2.18202977374 1.5453374847 -2.52414462864" /> -->
-             <!-- joana convert euler_from_quaternion 23 after intrisic calibration NOT BAD IN X
-              -->
-            <!-- <origin
-                xyz="0.250037605295 0.121920055033 -0.0198234097631"
-                rpy="1.86250666619 1.54643427609 -2.85870201824" /> -->
-             <!-- joana convert euler_from_quaternion 24 after intrisic calibration BEST ONE SO FAR i Y x: 0.337196  y: 0.190538
-              -->
-            <!-- <origin
-                xyz="0.249315737631 0.122836898871 -0.0173595499696"
-                rpy="1.94636293657 1.54585698373 -2.77753500665" /> -->
-             <!-- joana convert euler_from_quaternion 25 after intrisic calibration BAD In X
-              -->
-            <!-- <origin
-                xyz="0.2464362228 0.123022494194 -0.0186746162559"
-                rpy="1.94060142493 1.55129148344 -2.77733685521" /> -->
-             <!-- joana convert euler_from_quaternion 26 after intrisic calibration x: 0.333624  y: 0.193778
-              -->
-            <!-- <origin
-                xyz="0.279827354527 0.12116330125 -0.0182204436316"
-                rpy="1.78482730575 1.55059462639 -2.93123755032" /> -->
-             <!-- joana convert euler_from_quaternion 27 after intrisic calibration x: 0.33612 y: 0.191305
-              -->
-            <!-- <origin
-                xyz="0.247888432512 0.123172523076 -0.0197941758473"
-                rpy="1.90546337967 1.55051949778 -2.80537480944" /> -->
-             <!-- joana convert euler_from_quaternion 28 after intrisic calibration x: 0.333241 y: 0.191324 BEST SO FAR
-              -->
-            <!-- <origin
-                xyz="0.244316235557 0.128274081521 -0.0171762659762"
-                rpy="2.20778889637 1.54928707453 -2.49841856116" /> -->
-             <!-- joana convert euler_from_quaternion 29 after intrisic calibration BAD x: 0.305953 y: 0.19183
-              -->
-            <!-- <origin
-                xyz="0.24973940062 0.122363137841 -0.0173974204673"
-                rpy="1.95908118839 1.54394351042 -2.77092726247" /> -->
-             <!-- joana convert euler_from_quaternion 30 after intrisic calibration SOOO BAD x: 0.366387 y: 0.195049
-              -->
-            <!-- <origin
-                xyz="0.27831321288 0.125011986708 -0.0184730486361"
-                rpy="2.0482106047 1.54868496736 -2.65998966417" /> -->
-             <!-- joana convert euler_from_quaternion 31 after intrisic calibration SOOO x: 0.337417  y: 0.190311
-              -->
-            <!-- <origin
-                xyz="0.248760043608 0.120732900165 -0.0200442441181"
-                rpy="1.8905007158 1.54731656982 -2.84068026775" /> -->
-                <!-- x: 0.333534  y: 0.190602 -->
-<!-- x: 0.332586 y: 0.190537 -->
-            <!-- <origin
-                xyz="0.245460043608 0.120032900165 -0.0200442441181"
-                rpy="1.8905007158 1.54731656982 -2.84068026775" /> -->
              <!-- After Visions class X verry good x:0.330293 Y BAD y:0.199388    -->
             <!-- <origin
@@ -179,11 +16,59 @@
                 rpy="-1.16471837775 1.56523311718 0.4010175495" /> -->
              <!-- After Visions class X verry good x:0.330293 Y BAD y:0.199388    -->
+            <!-- <origin
+                xyz="0.247469111314 0.121665921033 -0.0209441353601"
+                rpy="-1.73229551223 1.56538317963 -0.168783829812" /> -->
+             <!-- After Visions class X verry good x:0.334 Y BAD y:0.195    -->
+            <!-- <origin
+                xyz="0.246027243916 0.123698162921 -0.0217020720854"
+                rpy="-2.08465796645 1.56316258117 -0.51351285704" /> -->
+             <!-- After Visions class X verry Bad   x: 0.335595  y: 0.197092 -->
+            <!-- <origin
+                xyz="0.279701284349 0.120790055045 -0.0218256377425"
+                rpy="-1.45806785305 1.56396145711 0.108188416383" /> -->
+             <!-- After Visions class X verry Bad   x: 0.309  y: 0.194 -->
+            <!-- <origin
+                xyz="0.248302667803 0.116857146075 -0.0200601728922"
+                rpy="-0.344850120367 1.56341182063 1.20453906713" /> -->
+             <!-- After Visions class X verry Bad  x: 0.336117  y: 0.196357 -->
+            <!-- <origin
+                xyz="0.248185448612 0.125125454595 -0.0200843255582"
+                rpy="-2.38753667624 1.56620697644 -0.824028438096" /> -->
+             <!-- After Visions class X verry Bad  x: 0.337626  y: 0.187725 -->
+            <!-- <origin
+                xyz="0.250665005218 0.113460975328 -0.0160878898623"
+                rpy="0.300623743189 1.56621707328 1.83520171316" /> -->
+             <!-- After Visions class X verry Bad  x: 0.333275  y: 0.189395 -->
+            <!-- <origin
+                xyz="0.246027243916 0.114460975328 -0.0160878898623"
+                rpy="0.300623743189 1.56621707328 1.83520171316" /> -->
+             <!-- After Visions class X verry Bad x: 0.333779  y: 0.191524 -->
+            <!-- <origin
+                xyz="0.246027243916 0.114460975328 -0.0160878898623"
+                rpy="-0.5940411655 1.56143330405 0.976778156421" /> -->
+             <!-- After Visions class X verry Bad  x: 0.335904  y: 0.195349 -->
+            <!-- <origin
+                xyz="0.248036425169 0.11731055525 -0.0227873939643"
+                rpy="-0.888625605858 1.56465194539 0.663431270648" /> -->
+             <!-- After Visions class X verry Bad  x: 0.335904  y: 0.195349 -->
+            <!-- <origin
+                xyz="0.247753167311 0.117209715472 -0.0211379268936"
+                rpy="-0.5940411655 1.56143330405 0.976778156421" /> -->
+             <!-- After Visions class X verry Bad  x: 0.335904  y: 0.195349 -->
+            <!-- <origin
+                xyz="0.245902887069 0.122097650666 -0.0210615785857"
+                rpy="-1.94792098497 1.56412947012 -0.385098127041" /> -->
+             <!-- After Visions class X verry Bad  x: 0.33381  y: 0.190073 -->
+            <!-- <origin
+                xyz="0.245525842462 0.115779043096 -0.017838428638"
+                rpy="-1.24022884812 1.5657875395 0.312412981998" /> -->
+             <!-- After Visions class X verry Bad  x: 0.330733  y: 0.190187 BEST  -->
             <origin
-                xyz="0.247469111314 0.121665921033 -0.0209441353601"
-                rpy="-1.73229551223 1.56538317963 -0.168783829812" />
-                <!--
-                X pouco menor 0.247998706401
-                Y menor 0.121920055033
-                 -->
+                xyz="0.242425842462 0.115779043096 -0.017838428638"
+                rpy="-1.24022884812 1.5657875395 0.312412981998" />
+             <!-- After Visions class X verry Bad  x: 0.3303 mas tambem pode ser 328.8  y: 0.190187 -->
+            <!-- <origin
+                xyz="0.242025842462 0.115779043096 -0.017838428638"
+                rpy="-1.24022884812 1.5657875395 0.312412981998" /> -->
         </xacro:kinect_camera>
     </xacro:macro>

File: bin_picking/urdf/binpicking_robot_macro.xacro (robot description, xacro)
@@ -24,5 +24,5 @@
         <xacro:bin_picking_sensor prefix="${prefix}ls_" />
         <joint name="${prefix}eef_tool_tip-${prefix}ls_base_link" type="fixed">
-            <origin xyz="0.0478 0.0166 -0.0636" rpy="0 0 0" />
+            <origin xyz="0 0 0" rpy="0 0 0" />
             <parent link="${prefix}eef_tool_tip" />
             <child link="${prefix}ls_base_link" />

File: bin_picking/urdf/binpicking_sensor_macro.xacro (robot description, xacro)
@@ -3,5 +3,11 @@
     xmlns:xacro="http://ros.org/wiki/xacro">
     <xacro:macro name="bin_picking_sensor" params="prefix">
-        <link name="${prefix}base_link">
+        <link name="${prefix}base_link" />
+        <joint name="${prefix}base_link-${prefix}optical_frame" type="fixed">
+            <origin xyz="0.0478 0.0166 -0.0636" rpy="0 0 0" />
+            <parent link="${prefix}base_link" />
+            <child link="${prefix}optical_frame" />
+        </joint>
+        <link name="${prefix}optical_frame">
             <visual>
                 <origin rpy="0 ${-pi/2} ${-pi}" xyz="-0.01215 0.0135 -0.0541" />
@@ -19,10 +25,4 @@
             </collision>
         </link>
-        <link name="${prefix}optical_frame" />
-        <joint name="${prefix}base_link-${prefix}optical_frame" type="fixed">
-            <origin xyz="0 0 0" rpy="0 0 0" />
-            <parent link="${prefix}base_link" />
-            <child link="${prefix}optical_frame" />
-        </joint>
     </xacro:macro>
 </robot>
