Commit message: beginning of kinect calibration

File: bin_picking/urdf/binpicking_sensor_macro.xacro (robot description, xacro)
@@ -5,5 +5,4 @@
         <link name="${prefix}base_link">
             <visual>
-                <!-- <origin rpy="0 0 0" xyz="0 0 0" /> -->
                 <origin rpy="0 ${-pi/2} ${-pi}" xyz="-0.01215 0.0135 -0.0541" />
                 <geometry>
@@ -15,5 +14,4 @@
             </visual>
             <collision>
-                <!-- <origin rpy="0 0 0" xyz="-0.16250 -0.03750 -0.03750"/> -->
                 <geometry>
                     <mesh filename="package://bin_picking/meshes/sensor.stl" />

Commit message: detection of the end-effcetor position for laser reading is now correct

File: bin_picking/urdf/binpicking_sensor_macro.xacro (robot description, xacro)
@@ -6,4 +6,5 @@
         <joint name="${prefix}base_link-${prefix}optical_frame" type="fixed">
             <origin xyz="0.0478 0.0166 -0.0636" rpy="0 0 0" />
+            <!-- <origin xyz="0.0478 0.0166 -0.0646" rpy="0 0 0" /> -->
             <parent link="${prefix}base_link" />
             <child link="${prefix}optical_frame" />
