Commit message: changes in organization

File: bin_picking/urdf/binpicking_gripper_macro.xacro (robot description, xacro)
@@ -2,5 +2,5 @@
 <robot
     xmlns:xacro="http://ros.org/wiki/xacro">
-    <xacro:property name="length" value="0.166" />
+    <xacro:property name="length" value="0.1675" />
     <xacro:property name="radius1" value="0.020" />
     <xacro:property name="radius2" value="0.007" />

Commit message: final alterations

File: bin_picking/urdf/binpicking_gripper_macro.xacro (robot description, xacro)
@@ -2,5 +2,5 @@
 <robot
     xmlns:xacro="http://ros.org/wiki/xacro">
-    <xacro:property name="length" value="0.1675" />
+    <xacro:property name="length" value="0.1640" />
     <xacro:property name="radius1" value="0.020" />
     <xacro:property name="radius2" value="0.007" />
